File: lumberjack.kicad_pcb (KiCad board)
At the start: 2 copper layers, 285.4 x 94.9 mm, 153 parts, among them J1 USB, J2 AVR_ISP_6, J3 JST, SW1 RESET, SW2 BOOT, U1 ATMEGA328-PU, Y1 16MHz

Commit message: WIP
Parts:
- removed J1: USB, lumberjack:USB_Mini-B
- removed REF**: OSHW-Logo2_9.8x8mm_Copper, Symbol:OSHW-Logo2_9.8x8mm_Copper
- added R5: 5.1k, Resistor_THT:R_Axial_DIN0204_L3.6mm_D1.6mm_P7.62mm_Horizontal, F.Cu at (37.8, 49.3)
- added R6: 5.1k, Resistor_THT:R_Axial_DIN0204_L3.6mm_D1.6mm_P7.62mm_Horizontal, F.Cu at (37.8, 52.5)
- added USB1: Type-C_USB_C_GCT_USB4085, lumberjack:USB_C_GCT_USB4085, F.Cu at (28.1, 54.8)
Connections:
- U1 pad 21: Net-(U1-Pad21) -> (no net)
Routing:
- net Net-(D67-Pad1): track 191.4 -> 171.7 mm
- net Net-(D66-Pad1): track 186.6 -> 175.0 mm
- net Net-(F1-Pad1): track 164.8 -> 155.3 mm
- net Net-(D1-Pad2): track 112.7 -> 113.9 mm
